File: schematics/System Block Diagram/System Block Diagram.kicad_sch (KiCad schematic)
At the start: 0 parts

Commit message: ..
Other:
- note added: "Database (PostgreSQL)"
- note added: "LoRaWAN module + piHat"
- note removed: "Database"
- note removed: "LoRaWAN piHat"
Changed lines of the file:
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@@
 	(rectangle
 		(start 178.816 119.761)
-		(end 195.326 123.571)
+		(end 205.105 123.571)
 		(stroke
 			(width 0)
@@
 	)
 	(rectangle
-		(start 197.485 143.764)
-		(end 209.296 148.971)
+		(start 189.611 144.399)
+		(end 201.422 149.606)
 		(stroke
 			(width 0)
@@
 	)
 	(rectangle
-		(start 176.276 117.856)
+		(start 176.276 118.11)
 		(end 215.646 152.781)
 		(stroke
@@
 	)
 	(rectangle
-		(start 182.626 133.985)
-		(end 192.151 140.97)
-		(stroke
-			(width 0)
-			(type default)
-		)
-		(fill
-			(type none)
-		)
-	)
-	(rectangle
-		(start 182.88 145.034)
-		(end 192.405 147.574)
+		(start 190.5 129.159)
+		(end 200.025 136.144)
+		(stroke
+			(width 0)
+			(type default)
+		)
+		(fill
+			(type none)
+		)
+	)
+	(rectangle
+		(start 188.722 137.541)
+		(end 201.422 142.621)
 		(stroke
 			(width 0)
@@
 		)
 	)
-	(text "Database"
-		(exclude_from_sim no)
-		(at 187.706 146.431 0)
+	(text "Database\n(PostgreSQL)"
+		(exclude_from_sim no)
+		(at 194.945 140.335 0)
 		(effects
 			(font
@@
 	(text "Dashboard\nSoftware"
 		(exclude_from_sim no)
-		(at 203.454 146.685 0)
-		(effects
-			(font
-				(size 1.27 1.27)
-			)
-		)
-	)
-	(text "LoRaWAN piHat"
-		(exclude_from_sim no)
-		(at 187.071 121.666 0)
+		(at 195.58 147.32 0)
+		(effects
+			(font
+				(size 1.27 1.27)
+			)
+		)
+	)
+	(text "LoRaWAN module + piHat"
+		(exclude_from_sim no)
+		(at 191.77 121.92 0)
 		(effects
 			(font
@@
 	(text "LoRaWAN \nNetwork \nManager"
 		(exclude_from_sim no)
-		(at 187.706 137.541 0)
+		(at 195.58 132.715 0)
 		(effects
 			(font
@@
 	(polyline
 		(pts
+			(xy 84.455 116.84) (xy 85.09 116.205)
+		)
+		(stroke
+			(width 0)
+			(type default)
+		)
+	)
+	(polyline
+		(pts
 			(xy 92.71 82.677) (xy 91.44 81.407)
 		)
@@
 		)
 		(stroke
+			(width 0)
+			(type default)
+		)
+	)
+	(polyline
+		(pts
+			(xy 83.82 116.205) (xy 84.455 116.84)
+		)
+		(stroke

Commit message: Final changes to pcbs before ordering
Other:
- note added: "Irrigation Actuator"
- note added: "LoRa"
- note removed: "Irrigation Controller"
Changed lines of the file:
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@@
 	)
 	(arc
-		(start 244.79 20.635)
-		(mid 247.6926 23.1524)
-		(end 247.965 26.985)
+		(start 244.729 32.004)
+		(mid 247.6316 34.5214)
+		(end 247.904 38.354)
 		(stroke
 			(width 0)
@@
 	)
 	(arc
-		(start 104.14 41.402)
-		(mid 107.4916 44.1054)
-		(end 107.95 48.387)
-		(stroke
-			(width 0)
-			(type default)
-		)
-		(fill
-			(type none)
-		)
-	)
-	(rectangle
-		(start 104.14 45.847)
-		(end 104.14 45.847)
-		(stroke
-			(width 0)
-			(type default)
-		)
-		(fill
-			(type none)
-		)
-	)
-	(arc
-		(start 245.425 23.175)
-		(mid 246.4545 23.8645)
-		(end 246.695 25.08)
+		(start 104.394 51.689)
+		(mid 107.7456 54.3924)
+		(end 108.204 58.674)
+		(stroke
+			(width 0)
+			(type default)
+		)
+		(fill
+			(type none)
+		)
+	)
+	(rectangle
+		(start 104.394 56.134)
+		(end 104.394 56.134)
+		(stroke
+			(width 0)
+			(type default)
+		)
+		(fill
+			(type none)
+		)
+	)
+	(arc
+		(start 245.364 34.544)
+		(mid 246.3935 35.2335)
+		(end 246.634 36.449)
 		(stroke
 			(width 0)
@@
 	)
 	(arc
-		(start 245.425 20)
-		(mid 248.7766 22.7034)
-		(end 249.235 26.985)
+		(start 245.364 31.369)
+		(mid 248.7156 34.0724)
+		(end 249.174 38.354)
 		(stroke
 			(width 0)
@@
 	)
 	(rectangle
-		(start 242.824 24.13)
+		(start 243.205 36.195)
 		(end 244.729 46.99)
 		(stroke
@@
 	)
 	(rectangle
-		(start 102.235 45.847)
+		(start 102.235 56.515)
 		(end 104.14 68.707)
 		(stroke
@@
 	)
 	(arc
-		(start 244.79 21.905)
-		(mid 246.9806 23.6014)
-		(end 247.33 26.35)
+		(start 244.729 33.274)
+		(mid 246.9196 34.9704)
+		(end 247.269 37.719)
 		(stroke
 			(width 0)
@@
 	)
 	(arc
-		(start 103.505 43.307)
-		(mid 105.6956 45.0034)
-		(end 106.045 47.752)
-		(stroke
-			(width 0)
-			(type default)
-		)
-		(fill
-			(type none)
-		)
-	)
-	(arc
-		(start 103.505 42.037)
-		(mid 106.4076 44.5544)
-		(end 106.68 48.387)
-		(stroke
-			(width 0)
-			(type default)
-		)
-		(fill
-			(type none)
-		)
-	)
-	(arc
-		(start 104.14 44.577)
-		(mid 105.1695 45.2665)
-		(end 105.41 46.482)
+		(start 103.759 53.594)
+		(mid 105.9496 55.2904)
+		(end 106.299 58.039)
+		(stroke
+			(width 0)
+			(type default)
+		)
+		(fill
+			(type none)
+		)
+	)
+	(arc
+		(start 103.759 52.324)
+		(mid 106.6616 54.8414)
+		(end 106.934 58.674)
+		(stroke
+			(width 0)
+			(type default)
+		)
+		(fill
+			(type none)
+		)
+	)
+	(arc
+		(start 104.394 54.864)
+		(mid 105.4235 55.5535)
+		(end 105.664 56.769)
 		(stroke
 			(width 0)
@@
 	(text "Sensor Node\n"
 		(exclude_from_sim no)
-		(at 88.138 55.626 0)
+		(at 74.422 56.896 0)
 		(effects
 			(font
@@
 		)
 	)
-	(text "Irrigation Controller"
+	(text "Irrigation Actuator"
 		(exclude_from_sim no)
 		(at 185.674 39.624 0)
@@
 		)
 	)
-	(text "LoRaWAN"
-		(exclude_from_sim no)
-		(at 103.886 39.878 0)
+	(text "LoRa\n"
+		(exclude_from_sim no)
+		(at 104.14 50.165 0)
 		(effects
 			(font
@@
 		)
 	)
-	(text "LoRaWAN"
-		(exclude_from_sim no)
-		(at 245.171 18.476 0)
-		(effects
-			(font
+	(text "LoRa"
+		(exclude_from_sim no)
+		(at 245.11 29.845 0)
+		(effects
+			(font
